File: pcb/aquarium.computer.brd (EAGLE design)
At the start: 112.6 x 74.3 mm, 55 parts, among them K1 JS-M1-9V-4, K2 JS-M1-9V-4, Q1 BC447, Q2 BC447, Q3 BC447, Q4 BC447, Q5 BC447, Q6 BC447, Q8 CSM-7X-DU, Q9 MC-306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

Commit message: rename
Parts:
- removed JP4: (no value), pinhead:1X02
- removed Q8: CSM-7X-DU, quarz:CSM-7X-DU
- removed R21: THERMISTOR-2,5, varistor:RS-2,5
- removed U$1: 4DIGITS-7SEGMENT-C, display-kingbright:CC56-12EWA
- removed U$3, U$4, U$5: PBS-18, switch:PBS18
- added 16MHZ: CSM-7X-DU, quarz:CSM-7X-DU
- added 7SEG: 4DIGITS-7SEGMENT-C, display-kingbright:CC56-12EWA
- added B1, B2, B3: PBS-18, switch:PBS18
- added D1: ES2D, diode:SMB
- added JP5: (no value), pinhead:1X03
- added TH1: THERMISTOR-2,5, varistor:RS-2,5
- moved X1 2.48 mm to (94.3, 39.1)
- moved JP1 2.29 mm to (49.9, 61.0)
- moved C6 1.60 mm to (64.5, 29.3)
- moved R5 0.91 mm to (44.9, 22.3)
- moved C3 0.85 mm to (64.5, 33.6)
- moved X3 0.48 mm to (14.4, 4.60), turned to 0 degrees
- moved R8 0.24 mm to (58.6, 38.7)
- renumbered JP2 to ISP, Q9 to 32.768K, U$2 to BAT, U1 to M328, U2 to RTC
Connections:
- new net N$74: D1.A, X1.1
- net GND: now also B1.A, B2.A, B3.A, JP5.3; no longer JP4.2, U$3.A, U$4.A, U$5.A
- net N$12: now also X3.1; no longer X3.2
- net N$30: now also 16MHZ.2; no longer Q8.2
- net N$31: now also 16MHZ.1; no longer Q8.1
- net N$32: now also 7SEG.11; no longer U$1.11
- net N$36: now also TH1.2; no longer R21.2
- net N$44: now also 7SEG.7; no longer U$1.7
- net N$49: now also B2.B; no longer U$4.B
- net N$50: now also B1.B; no longer U$3.B
- net N$51: now also B3.B; no longer U$5.B
- net N$52: now also 7SEG.10; no longer U$1.10
- net N$53: now also 7SEG.4; no longer U$1.4
- net N$54: now also 7SEG.2; no longer U$1.2
- net N$55: now also 7SEG.1; no longer U$1.1
- net N$56: now also 7SEG.5; no longer U$1.5
- net N$57: now also 7SEG.6; no longer U$1.6
- net N$58: now also 7SEG.12; no longer U$1.12
- net N$59: now also 7SEG.9; no longer U$1.9
- net N$60: now also 7SEG.8; no longer U$1.8
- net N$61: now also 7SEG.3; no longer U$1.3
- net N$68: now also JP5.1; no longer JP4.1
- net N$73: now also D1.C, X3.2; no longer X1.1, X3.1
- net VCC: now also JP5.2, TH1.1; no longer R21.1
Routing:
- net VCC: track 156.9 -> 108.4 mm
- net N$74: track 0.00 -> 6.16 mm
- net N$30: track 13.9 -> 19.0 mm
- net GND: track 268.7 -> 263.9 mm, vias 3 -> 2
- net N$31: track 8.36 -> 12.8 mm
- net N$27: track 46.0 -> 43.2 mm
- net N$73: track 123.1 -> 121.1 mm
- net N$26: track 43.7 -> 41.9 mm
- net N$10: track 30.7 -> 29.2 mm
- net N$9: track 29.7 -> 28.3 mm
- net N$36: track 46.7 -> 45.2 mm
- net N$8: track 29.6 -> 28.3 mm
- net N$2: track 23.5 -> 24.6 mm
- net N$14: track 24.0 -> 25.0 mm
- net N$25: track 41.8 -> 40.9 mm
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Other:
- board size 112.6 x 74.3 mm -> 112.5 x 75.6 mm
- board text added: "+"
- board text added: "+12V"
- board text added: "+5V"
- board text added: "D"
- board text added: "GND"
- board text added: "LM1117"
- board text added: "N"

Commit message: thermistor code
Parts:
- C1, C2: value (none) -> 100n
- C5: value (none) -> 10uF
- R1, R2, R3, R4, R5, R6: value (none) -> 4k7
- R10, R11, R12, R13, R14, R15, R16, R9: value (none) -> 330
- R17, R18, R7, R8: value (none) -> 10k
